Commit message: Update tb4_description for sim

File: nav2_minimal_turtlebot_simulation/nav2_minimal_tb4_description/urdf/icreate/caster_mir.urdf.xacro (robot description, xacro)
@@ -28,5 +28,5 @@
     <preserveFixedJoint>true</preserveFixedJoint>
   </gazebo>
-  <gazebo reference="${name}_link">
+  <!-- <gazebo reference="${name}_link">
     <material>Gazebo/DarkGrey</material>
     <mu1>0.1</mu1>
@@ -34,4 +34,11 @@
     <kp>1000000.0</kp>
     <kd>1.0</kd>
+  </gazebo> -->
+  <gazebo reference="${name}_link">
+    <material>Gazebo/DarkGrey</material>
+    <mu1>100.0</mu1>
+    <mu2>100.0</mu2>
+    <kp>100000.0</kp>
+    <kd>10.0</kd>
   </gazebo>
 </xacro:macro>

File: nav2_minimal_turtlebot_simulation/nav2_minimal_tb4_description/urdf/standard/turtlebot4_1liadrs.urdf.xacro (robot description, xacro)
@@ -13,6 +13,5 @@
     <visual>
       <geometry>
-        <!-- <box size="0.5 0.3 0.2"/> -->
-        <box size="0.65 0.65 0.2"/>
+        <box size="0.5 0.3 0.2"/>
       </geometry>
       <material name="light_grey">
@@ -22,6 +21,5 @@
     <collision>
       <geometry>
-        <!-- <box size="0.5 0.3 0.2"/> -->
-        <box size="0.65 0.65 0.2"/>
+        <box size="0.5 0.3 0.2"/>
       </geometry>
     </collision>

File: nav2_minimal_turtlebot_simulation/nav2_minimal_tb4_description/urdf/standard/turtlebot4_2liadrs.urdf.xacro (robot description, xacro)
@@ -12,17 +12,9 @@
   <link name="chassis_link">
     <visual>
-      <geometry>
-        <!-- <box size="0.5 0.3 0.2"/> -->
-        <box size="0.65 0.65 0.2"/>
-      </geometry>
-      <material name="light_grey">
-        <color rgba="0.8 0.8 0.8 1.0"/>
-      </material>
+      <box size="0.5 0.3 0.2"/>
+      <material name="light_grey"><color rgba="0.8 0.8 0.8 1.0"/></material>
     </visual>
     <collision>
-      <geometry>
-        <!-- <box size="0.5 0.3 0.2"/> -->
-        <box size="0.65 0.65 0.2"/>
-      </geometry>
+      <geometry><box size="0.5 0.3 0.2"/></geometry>
     </collision>
     <!-- <inertial>
@@ -41,8 +33,13 @@
     <parent link="base_link"/>
     <child link="chassis_link"/>
-    <origin xyz="0 0 0.15" rpy="0 0 0"/>
+    <origin xyz="0 0 0.05" rpy="0 0 0"/>
   </joint>
-  <xacro:rplidar name="rplidar" parent_link="chassis_link" gazebo="$(arg gazebo)">
-    <origin xyz="0.0 0.0 0.15" rpy="0 0 0"/>
+  <xacro:rplidar name="front_rplidar" parent_link="chassis_link" gazebo="$(arg gazebo)">
+    <origin xyz="0.20 0.10 0.12" rpy="0 0 ${0.25 * 3.14159}" />
+    <xacro:property name="topic" value="front_scan" />
+  </xacro:rplidar>
+  <xacro:rplidar name="back_rplidar" parent_link="chassis_link" gazebo="$(arg gazebo)">
+    <origin xyz="-0.20 -0.10 0.12" rpy="0 0 ${-0.75 * 3.14159}" />
+    <xacro:property name="topic" value="back_scan" />
   </xacro:rplidar>
   <xacro:oakd model="pro" parent_link="chassis_link">
